File: rpi-ledarray-eagle.brd (EAGLE design)
At the start: 33.1 x 15.8 mm, 21 parts

Commit message: Added OSHW logo. Added rev number on the bottom copper. Increased resistor silk label size.
Parts:
- added U$2: (no value), ohw-logo:OSHW_FILLX200_NOTEXT
Other:
- board text added: "R. Nugent prizepony.us"
- board text added: "Rev1"
- board text removed: "R. Nugent prizepony.us 2013"
