File: rpi-ledarray-eagle.sch (EAGLE design)
At the start: 27 parts

Commit message: First version finished
Parts:
- removed LED11, LED12, LED13: (no value), SparkFun:LED1206
- removed R11, R12, R13, R14, R15, R16, R17: 270, SparkFun:RESISTOR1206
- added R1, R10, R2, R9: (no value), SparkFun:RESISTOR1206
- R3, R4, R5, R6, R7, R8: value 270 -> (none)
Connections:
- removed net N$16: LED12.A, R16.2
- removed net N$17: LED13.A, R17.2
- removed net N$7: LED5.A, R7.2
- removed net N$8: LED6.A, R8.2
- new net 3V3_1: JP1.1
- new net 3V3_2: JP1.17
- new net N$10: LED10.A, R10.2
- net 5V: now also R1.1, R10.1, R2.1, R9.1; no longer R11.1, R12.1, R13.1, R14.1, R15.1, R16.1, R17.1
- net GPIO10_MOSI: no longer LED5.C
- net GPIO11_SCLK: no longer LED6.C
- net GPIO17: now also LED2.C; no longer LED7.C
- net GPIO18: now also LED5.C; no longer LED8.C
- net GPIO22: now also LED4.C; no longer LED9.C
- net GPIO23: now also LED6.C; no longer LED10.C
- net GPIO24: now also LED7.C; no longer LED11.C
- net GPIO25: now also LED8.C; no longer LED12.C
- net GPIO27: now also LED3.C; no longer LED13.C
- net GPIO7: now also LED10.C; no longer LED2.C
- net GPIO8: now also LED9.C; no longer LED3.C
- net GPIO9_MISO: no longer LED4.C
- net N$11: now also LED9.A, R9.2; no longer LED7.A, R11.2
- net N$12: now also R8.2; no longer R12.2
- net N$13: now also LED7.A, R7.2; no longer LED9.A, R13.2
- net N$14: now also LED6.A, R6.2; no longer LED10.A, R14.2
- net N$15: now also LED5.A, R5.2; no longer LED11.A, R15.2
- net N$3: now also R1.2; no longer R3.2
- net N$4: now also R3.2; no longer R5.2
- net N$5: now also R2.2; no longer R4.2
- net N$6: now also R4.2; no longer R6.2
Other:
- moved on the sheet: JP1, LED1, LED10, LED2, LED3, LED4, LED5, LED6, LED7, LED8, LED9, R3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

Commit message: Changed resistors to 0603. Shrunk the board dimensions.
Parts:
- R1, R10, R2, R3, R4, R5, R6, R7, R8, R9: device SparkFun:RESISTOR1206 -> SparkFun:RESISTOR0603-RES
